Commit message: Changes to merge

File: quad_description/urdf/kit_c.urdf (robot description, URDF)
Before this commit: robot quad, 6 links, 5 joints
Links:
- link base_link_inertia: geometry collision box size=1 1 0.5; visual mesh filename=package://rotors_description/meshes/hummingbird.dae scale=1 1 1

File: quad_description/urdf/kit_c.xacro (robot description, xacro)
@@ -87,5 +87,5 @@
     mesh ="propeller"
     mesh_scale="${mesh_scale_prop}"
-    color="Grey">
+    color="Red">
     <origin xyz="0 -${arm_length} ${rotor_offset_top}" rpy="0 0 0" />
     <xacro:insert_block name="rotor_inertia" />
@@ -108,5 +108,5 @@
     mesh ="propeller"
     mesh_scale="${mesh_scale_prop}"
-    color="Grey">
+    color="Green">
     <origin xyz="-${arm_length} 0 ${rotor_offset_top}" rpy="0 0 0" />
     <xacro:insert_block name="rotor_inertia" />
@@ -129,5 +129,5 @@
     mesh ="propeller"
     mesh_scale="${mesh_scale_prop}"
-    color="Grey">
+    color="Yellow">
     <origin xyz="0 ${arm_length} ${rotor_offset_top}" rpy="0 0 0" />
     <xacro:insert_block name="rotor_inertia" />
