Commit message: Embedding preparations

File: quad_description/urdf/component_snippets.xacro (robot description, xacro)
@@ -25,6 +25,6 @@
         <robotNamespace>${namespace}</robotNamespace>
         <bagFileName>${bag_file}</bagFileName>
-        <linkName>base_link</linkName>
-        <frameId>base_link</frameId>
+        <linkName>cam0</linkName>
+        <frameId>cam0</frameId>
         <commandAttitudeThrustSubTopic>command/attitude</commandAttitudeThrustSubTopic>
         <commandAttitudeThrustPubTopic>command/attitude</commandAttitudeThrustPubTopic>
@@ -188,5 +188,5 @@
     <gazebo>
       <plugin filename="librotors_gazebo_odometry_plugin.so" name="odometry_sensor${odometry_sensor_suffix}">
-        <linkName>base_link</linkName>  <!--{namespace}/odometry_sensor${odometry_sensor_suffix}_link"-->
+        <linkName>cam0</linkName>  <!--{namespace}/odometry_sensor${odometry_sensor_suffix}_link"-->
         <robotNamespace>${namespace}</robotNamespace>
         <poseTopic>${pose_topic}</poseTopic>
@@ -221,6 +221,6 @@
     <gazebo>
       <plugin filename="librotors_gazebo_wind_plugin.so" name="wind_plugin">
-        <frameId>base_link</frameId>
-        <linkName>base_link</linkName>
+        <frameId>cam0</frameId>
+        <linkName>cam0</linkName>
         <robotNamespace>${namespace}</robotNamespace>
         <xyzOffset>${xyz_offset}</xyzOffset> <!-- [m] [m] [m] -->

File: quad_description/urdf/iris.xacro (robot description, xacro)
@@ -61,5 +61,5 @@
     motor_constant="${motor_constant}"
     moment_constant="${moment_constant}"
-    parent="base_link"
+    parent="cam0"
     mass_rotor="${mass_rotor}"
     radius_rotor="${radius_rotor}"
@@ -82,5 +82,5 @@
     motor_constant="${motor_constant}"
     moment_constant="${moment_constant}"
-    parent="base_link"
+    parent="cam0"
     mass_rotor="${mass_rotor}"
     radius_rotor="${radius_rotor}"
@@ -102,5 +102,5 @@
     motor_constant="${motor_constant}"
     moment_constant="${moment_constant}"
-    parent="base_link"
+    parent="cam0"
     mass_rotor="${mass_rotor}"
     radius_rotor="${radius_rotor}"
@@ -122,5 +122,5 @@
     motor_constant="${motor_constant}"
     moment_constant="${moment_constant}"
-    parent="base_link"
+    parent="cam0"
     mass_rotor="${mass_rotor}"
     radius_rotor="${radius_rotor}"

File: quad_description/urdf/iris_base.xacro (robot description, xacro)
@@ -14,5 +14,5 @@
     namespace="${namespace}"
     imu_suffix=""
-    parent_link="base_link"
+    parent_link="cam0"
     imu_topic="imu"
     mass_imu_sensor="0.015"
@@ -34,5 +34,5 @@
       namespace="${namespace}"
       imu_suffix="gt"
-      parent_link="base_link"
+      parent_link="cam0"
       imu_topic="ground_truth/imu"
       mass_imu_sensor="0.00001"
@@ -53,5 +53,5 @@
       namespace="${namespace}/ground_truth"
       odometry_sensor_suffix="gt"
-      parent_link="base_link"
+      parent_link="cam0"
       pose_topic="pose"
       pose_with_covariance_topic="pose_with_covariance"

File: quad_description/urdf/kit_c.urdf (robot description, URDF)
Before this commit: robot quad, 6 links, 5 joints
Links:
- removed link base_link
- added link cam0
Joints:
- joint base_joint: parent base_link -> cam0
- joint rotor_0_joint: parent base_link -> cam0
- joint rotor_1_joint: parent base_link -> cam0
- joint rotor_2_joint: parent base_link -> cam0
- joint rotor_3_joint: parent base_link -> cam0

File: quad_description/urdf/kit_c.xacro (robot description, xacro)
@@ -55,5 +55,5 @@
     motor_constant="${motor_constant}"
     moment_constant="${moment_constant}"
-    parent="base_link"
+    parent="cam0"
     mass_rotor="${mass_rotor}"
     radius_rotor="${radius_rotor}"
@@ -76,5 +76,5 @@
     motor_constant="${motor_constant}"
     moment_constant="${moment_constant}"
-    parent="base_link"
+    parent="cam0"
     mass_rotor="${mass_rotor}"
     radius_rotor="${radius_rotor}"
@@ -97,5 +97,5 @@
     motor_constant="${motor_constant}"
     moment_constant="${moment_constant}"
-    parent="base_link"
+    parent="cam0"
     mass_rotor="${mass_rotor}"
     radius_rotor="${radius_rotor}"
@@ -118,5 +118,5 @@
     motor_constant="${motor_constant}"
     moment_constant="${moment_constant}"
-    parent="base_link"
+    parent="cam0"
     mass_rotor="${mass_rotor}"
     radius_rotor="${radius_rotor}"

File: quad_description/urdf/kit_c_base.xacro (robot description, xacro)
@@ -14,5 +14,5 @@
     namespace="${namespace}"
     imu_suffix=""
-    parent_link="base_link"
+    parent_link="cam0"
     imu_topic="imu"
     mass_imu_sensor="0.015"
@@ -33,5 +33,5 @@
     <xacro:camera_macro
       namespace="${namespace}"
-      parent_link="base_link"
+      parent_link="cam0"
       camera_suffix=""
       frame_rate="30"
@@ -54,5 +54,5 @@
     <xacro:vi_sensor_depth_macro
       namespace="${namespace}"
-      parent_link="base_link"
+      parent_link="cam0"
       camera_suffix=""
       frame_rate="30"
@@ -66,5 +66,5 @@
       namespace="${namespace}"
       imu_suffix="gt"
-      parent_link="base_link"
+      parent_link="cam0"
       imu_topic="ground_truth/imu"
       mass_imu_sensor="0.00001"
@@ -85,5 +85,5 @@
       namespace="${namespace}/ground_truth"
       odometry_sensor_suffix="gt"
-      parent_link="base_link"
+      parent_link="cam0"
       pose_topic="pose"
       pose_with_covariance_topic="pose_with_covariance"

File: quad_description/urdf/kit_c_kinect.xacro (robot description, xacro)
@@ -14,5 +14,5 @@
     namespace="${namespace}"
     imu_suffix=""
-    parent_link="base_link"
+    parent_link="cam0"
     imu_topic="imu"
     mass_imu_sensor="0.015"
@@ -32,5 +32,5 @@
     <xacro:vi_sensor_depth_macro
       namespace="${namespace}"
-      parent_link="base_link"
+      parent_link="cam0"
       camera_suffix=""
       frame_rate="30"
@@ -42,5 +42,5 @@
       namespace="${namespace}"
       imu_suffix="gt"
-      parent_link="base_link"
+      parent_link="cam0"
       imu_topic="ground_truth/imu"
       mass_imu_sensor="0.00001"
@@ -61,5 +61,5 @@
       namespace="${namespace}/ground_truth"
       odometry_sensor_suffix="gt"
-      parent_link="base_link"
+      parent_link="cam0"
       pose_topic="pose"
       pose_with_covariance_topic="pose_with_covariance"

File: quad_description/urdf/multirotor_base.xacro (robot description, xacro)
@@ -20,8 +20,8 @@
   <xacro:macro name="multirotor_base_macro"
     params="robot_namespace mass body_width body_height mesh_file mesh_scale color *inertia">
-    <link name="base_link"></link>
+    <link name="cam0"></link>
     <joint name="base_joint" type="fixed">
       <origin xyz="0 0 0" rpy="0 0 0" />
-      <parent link="base_link" />
+      <parent link="cam0" />
       <child link="base_link_inertia" />
     </joint>
@@ -47,13 +47,13 @@
       </collision>
     </link>
-    <!-- attach multirotor_base_plugin to the base_link -->
+    <!-- attach multirotor_base_plugin to the cam0 -->
     <gazebo>
       <plugin filename="librotors_gazebo_multirotor_base_plugin.so" name="rosbag">
         <robotNamespace>${robot_namespace}</robotNamespace>
-        <linkName>base_link</linkName>
+        <linkName>cam0</linkName>
         <rotorVelocitySlowdownSim>${rotor_velocity_slowdown_sim}</rotorVelocitySlowdownSim>
       </plugin>
     </gazebo>
-    <gazebo reference="base_link">
+    <gazebo reference="cam0">
       <material>Gazebo/${color}</material>
     </gazebo>

File: quad_description/urdf/sensors/static_camera.urdf.xacro (robot description, xacro)
@@ -13,5 +13,5 @@
   <xacro:macro name="camera_base_macro"
     params="robot_namespace mass body_width body_height *inertia">
-    <link name="base_link">
+    <link name="cam0">
       <!-- <collision> -->
         <!-- <origin xyz="0 0 0" rpy="0 0 0" /> -->
@@ -36,5 +36,5 @@
       <axis xyz="0 1 0" />
       <origin xyz="0 0 0" rpy="0 0 0" />
-      <parent link="base_link" />
+      <parent link="cam0" />
       <child link="camera_link" />
     </joint>
