Commit message: Lots of long overdue changes.

File: quad_description/urdf/kit_c_irl.xacro (robot description, xacro)
@@ -5,12 +5,11 @@
   <xacro:property name="mesh_file" value="hummingbird.dae" />
   <xacro:property name="mesh_scale" value="1 1 1"/>
-  <xacro:property name="mesh" value="propeller"/>  <!-- "propeller" -->
-  <xacro:property name="body_width" value="0.3" /> <!-- [m] -->
-  <xacro:property name="body_height" value="0.17" /> <!-- [m] -->
+  <xacro:property name="body_width" value="2" /> <!-- [m] -->
+  <xacro:property name="body_height" value="0.5" /> <!-- [m] -->
   <xacro:property name="color" value="DarkGrey" />
   <!-- Main multirotor link -->
   <xacro:macro name="multirotor_base_macro"
-    params="robot_namespace mass body_width body_height mesh_file mesh_scale color *inertia">
-    <link name="cam0"></link>
+    params="robot_namespace body_width body_height mesh_file mesh_scale color">
+    <link name="cam0">
       <visual>
         <origin xyz="0 0 0" rpy="0 0 0" />
@@ -32,5 +31,4 @@
   <xacro:multirotor_base_macro
     robot_namespace="${namespace}"
-    mass="${mass}"
     body_width="${body_width}"
     body_height="${body_height}"
@@ -38,5 +36,4 @@
     mesh_scale="${mesh_scale}"
     color="${color}">
-    <xacro:insert_block name="body_inertia" />
   </xacro:multirotor_base_macro>
 </robot>

Commit message: Perf param changes

File: quad_description/urdf/kit_c_irl.xacro (robot description, xacro)
@@ -5,5 +5,5 @@
   <xacro:property name="mesh_file" value="hummingbird.dae" />
   <xacro:property name="mesh_scale" value="1 1 1"/>
-  <xacro:property name="body_width" value="2" /> <!-- [m] -->
+  <xacro:property name="body_width" value="1" /> <!-- [m] -->
   <xacro:property name="body_height" value="0.5" /> <!-- [m] -->
   <xacro:property name="color" value="DarkGrey" />
